File: hardware/DashShield.kicad_sch (KiCad schematic)
At the start: 112 parts, among them J001 PWR, J101 CAN0, J202 CAN1, J3 Dash LEDs, J301 Steering Wheel, J601 GPIO, Q301 2N7002, Q302 2N7002, Q303 2N7002, Q501 2N7002, Q502 2N7002, Q503 2N7002, Q504 2N7002, Q505 2N7002, Q506 2N7002, U101 MCP2515-xST, U102 MCP2562-E-SN, U201 MCP2515-xST, U202 MCP2562-E-SN, U401 CAT24C256, Y101 8MHz, Y201 8MHz

Commit message: chore: upload progress
Parts:
- added H601, H602, H603, H604: MH, MountingHole:MountingHole_2.7mm_M2.5_Pad, symbol Mechanical:MountingHole
- C102, C103, C202, C203: value 22pF -> 16pF
- Y101, Y201: footprint Crystal:Crystal_SMD_HC49-SD -> Crystal:Crystal_C38-LF_D3.0mm_L8.0mm_Vertical
Changed lines of the file:
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@@
+    )
+  )
+  (symbol (lib_id "Mechanical:MountingHole") (at 96.52 27.94 0) (unit 1)
+    (in_bom yes) (on_board yes) (dnp no) (fields_autoplaced)
+    (property "Reference" "H604" (at 99.06 26.67 0)
+      (effects (font (size 1.27 1.27)) (justify left))
+    )
+    (property "Value" "MH" (at 99.06 29.21 0)
+      (effects (font (size 1.27 1.27)) (justify left))
+    )
+    (property "Footprint" "MountingHole:MountingHole_2.7mm_M2.5_Pad" (at 96.52 27.94 0)
+      (effects (font (size 1.27 1.27)) hide)
+    )
+    (property "Datasheet" "~" (at 96.52 27.94 0)
+      (effects (font (size 1.27 1.27)) hide)
+    )
+    (instances
+      (project "DashShield"
+        (path "/e63e39d7-6ac0-4ffd-8aa3-1841a4541b55"
+          (reference "H604") (unit 1)
+        )
+      )
+    )
+  )
+  (symbol (lib_id "Mechanical:MountingHole") (at 96.52 22.86 0) (unit 1)
+    (in_bom yes) (on_board yes) (dnp no) (fields_autoplaced)
+    (property "Reference" "H602" (at 99.06 21.59 0)
+      (effects (font (size 1.27 1.27)) (justify left))
+    )
+    (property "Value" "MH" (at 99.06 24.13 0)
+      (effects (font (size 1.27 1.27)) (justify left))
+    )
+    (property "Footprint" "MountingHole:MountingHole_2.7mm_M2.5_Pad" (at 96.52 22.86 0)
+      (effects (font (size 1.27 1.27)) hide)
+    )
+    (property "Datasheet" "~" (at 96.52 22.86 0)
+      (effects (font (size 1.27 1.27)) hide)
+    )
+    (instances
+      (project "DashShield"
+        (path "/e63e39d7-6ac0-4ffd-8aa3-1841a4541b55"
+          (reference "H602") (unit 1)
+        )
+      )
     )
   )
@@
     )
   )
+  (symbol (lib_id "Mechanical:MountingHole") (at 86.36 22.86 0) (unit 1)
+    (in_bom yes) (on_board yes) (dnp no) (fields_autoplaced)
+    (property "Reference" "H601" (at 88.9 21.59 0)
+      (effects (font (size 1.27 1.27)) (justify left))
+    )
+    (property "Value" "MH" (at 88.9 24.13 0)
+      (effects (font (size 1.27 1.27)) (justify left))
+    )
+    (property "Footprint" "MountingHole:MountingHole_2.7mm_M2.5_Pad" (at 86.36 22.86 0)
+      (effects (font (size 1.27 1.27)) hide)
+    )
+    (property "Datasheet" "~" (at 86.36 22.86 0)
+      (effects (font (size 1.27 1.27)) hide)
+    )
+    (instances
+      (project "DashShield"
+        (path "/e63e39d7-6ac0-4ffd-8aa3-1841a4541b55"
+          (reference "H601") (unit 1)
+        )
+      )
+    )
+  )
   (symbol (lib_id "Device:R") (at 363.22 55.88 90) (unit 1)
     (in_bom yes) (on_board yes) (dnp no)
@@
       (effects (font (size 1.27 1.27)))
     )
-    (property "Value" "22pF" (at 229.87 125.73 90)
+    (property "Value" "16pF" (at 229.87 125.73 90)
       (effects (font (size 1.27 1.27)))
     )
@@
       (effects (font (size 1.27 1.27)) (justify right))
     )
-    (property "Footprint" "Crystal:Crystal_SMD_HC49-SD" (at 237.49 134.62 0)
-      (effects (font (size 1.27 1.27)) hide)
-    )
-    (property "Datasheet" "https://abracon.com/Resonators/ABLS.pdf" (at 237.49 134.62 0)
+    (property "Footprint" "Crystal:Crystal_C38-LF_D3.0mm_L8.0mm_Vertical" (at 237.49 134.62 0)
+      (effects (font (size 1.27 1.27)) hide)
+    )
+    (property "Datasheet" "https://abracon.com/Resonators/ab308.pdf" (at 237.49 134.62 0)
       (effects (font (size 1.27 1.27)) hide)
     )
@@
       (effects (font (size 1.27 1.27)))
     )
-    (property "Value" "22pF" (at 229.87 59.69 90)
+    (property "Value" "16pF" (at 229.87 59.69 90)
       (effects (font (size 1.27 1.27)))
     )
@@
       (effects (font (size 1.27 1.27)) (justify right))
     )
-    (property "Footprint" "Crystal:Crystal_SMD_HC49-SD" (at 237.49 58.42 0)
-      (effects (font (size 1.27 1.27)) hide)
-    )
-    (property "Datasheet" "https://abracon.com/Resonators/ABLS.pdf" (at 237.49 58.42 0)
+    (property "Footprint" "Crystal:Crystal_C38-LF_D3.0mm_L8.0mm_Vertical" (at 237.49 58.42 0)
+      (effects (font (size 1.27 1.27)) hide)
+    )
+    (property "Datasheet" "https://abracon.com/Resonators/ab308.pdf" (at 237.49 58.42 0)
       (effects (font (size 1.27 1.27)) hide)
     )
@@
     )
   )
+  (symbol (lib_id "Mechanical:MountingHole") (at 86.36 27.94 0) (unit 1)
+    (in_bom yes) (on_board yes) (dnp no)
+    (property "Reference" "H603" (at 88.9 26.67 0)
+      (effects (font (size 1.27 1.27)) (justify left))
+    )
+    (property "Value" "MH" (at 88.9 29.21 0)
+      (effects (font (size 1.27 1.27)) (justify left))
+    )
+    (property "Footprint" "MountingHole:MountingHole_2.7mm_M2.5_Pad" (at 86.36 27.94 0)
+      (effects (font (size 1.27 1.27)) hide)
+    )
+    (property "Datasheet" "~" (at 86.36 27.94 0)
+      (effects (font (size 1.27 1.27)) hide)
+    )
+    (instances
+      (project "DashShield"
+        (path "/e63e39d7-6ac0-4ffd-8aa3-1841a4541b55"
+          (reference "H603") (unit 1)
+        )
+      )
+    )
+  )
   (symbol (lib_id "power:+3.3V") (at 46.99 166.37 0) (unit 1)
     (in_bom yes) (on_board yes) (dnp no)
@@
       (effects (font (size 1.27 1.27)))
     )
-    (property "Value" "22pF" (at 229.87 135.89 90)
+    (property "Value" "16pF" (at 229.87 135.89 90)
       (effects (font (size 1.27 1.27)))
     )
@@
       (effects (font (size 1.27 1.27)))
     )
-    (property "Value" "22pF" (at 229.87 49.53 90)
-      (effects (font (size 1.27 1.27)))
-    )
+    (property "Value" "16pF" (at 229.87 49.53 90)
+      (effects (font (size 1.27 1.27)))
+    )

Commit message: Chore-Upload progress
Parts:
- JP101, JP102, JP201, JP202: footprint Connector_PinHeader_2.54mm:PinHeader_1x02_P2.54mm_Vertical -> Jumper:SolderJumper-2_P1.3mm_Open_RoundedPad1.0x1.5mm; symbol Jumper:Jumper_2_Open -> Jumper:SolderJumper_2_Open
- JP401: renamed from JP1; footprint Connector_PinHeader_2.54mm:PinHeader_1x02_P2.54mm_Vertical -> Jumper:SolderJumper-2_P1.3mm_Open_RoundedPad1.0x1.5mm; symbol Jumper:Jumper_2_Open -> Jumper:SolderJumper_2_Open
Changed lines of the file:
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@@
     (stroke (width 0) (type default))
   )
-  (wire (pts (xy 367.03 132.08) (xy 370.84 132.08))
-    (stroke (width 0) (type default))
-  )
   (wire (pts (xy 342.9 128.27) (xy 342.9 129.54))
     (stroke (width 0) (type default))
@@
     (stroke (width 0) (type default))
   )
+  (wire (pts (xy 379.73 132.08) (xy 381 132.08))
+    (stroke (width 0) (type default))
+  )
   (wire (pts (xy 69.85 29.21) (xy 69.85 31.75))
     (stroke (width 0) (type solid))
@@
     (stroke (width 0) (type default))
   )
+  (wire (pts (xy 378.46 74.93) (xy 384.81 74.93))
+    (stroke (width 0) (type default))
+  )
   (wire (pts (xy 308.61 182.88) (xy 287.02 182.88))
     (stroke (width 0) (type default))
@@
     (stroke (width 0) (type default))
   )
-  (wire (pts (xy 384.81 151.13) (xy 379.73 151.13))
+  (wire (pts (xy 378.46 151.13) (xy 384.81 151.13))
     (stroke (width 0) (type default))
   )
@@
     (stroke (width 0) (type default))
   )
-  (wire (pts (xy 201.93 165.1) (xy 208.28 165.1))
+  (wire (pts (xy 200.66 165.1) (xy 208.28 165.1))
     (stroke (width 0) (type default))
   )
@@
     (stroke (width 0) (type default))
   )
-  (wire (pts (xy 379.73 74.93) (xy 384.81 74.93))
-    (stroke (width 0) (type default))
-  )
   (wire (pts (xy 194.31 143.51) (xy 186.69 143.51))
     (stroke (width 0) (type solid))
@@
     (stroke (width 0) (type default))
   )
-  (wire (pts (xy 367.03 55.88) (xy 370.84 55.88))
+  (wire (pts (xy 367.03 55.88) (xy 372.11 55.88))
     (stroke (width 0) (type default))
   )
@@
     (stroke (width 0) (type solid))
   )
-  (wire (pts (xy 342.9 151.13) (xy 369.57 151.13))
+  (wire (pts (xy 342.9 151.13) (xy 370.84 151.13))
     (stroke (width 0) (type default))
   )
@@
     (stroke (width 0) (type default))
   )
+  (wire (pts (xy 367.03 132.08) (xy 372.11 132.08))
+    (stroke (width 0) (type default))
+  )
   (wire (pts (xy 342.9 50.8) (xy 342.9 52.07))
     (stroke (width 0) (type default))
@@
     (stroke (width 0) (type default))
   )
-  (wire (pts (xy 342.9 74.93) (xy 369.57 74.93))
+  (wire (pts (xy 342.9 74.93) (xy 370.84 74.93))
     (stroke (width 0) (type default))
   )
@@
     (stroke (width 0) (type solid))
   )
+  (wire (pts (xy 379.73 55.88) (xy 381 55.88))
+    (stroke (width 0) (type default))
+  )
   (wire (pts (xy 157.48 111.76) (xy 165.1 111.76))
     (stroke (width 0) (type default))
@@
     (stroke (width 0) (type default))
   )
-  (wire (pts (xy 186.69 165.1) (xy 191.77 165.1))
+  (wire (pts (xy 186.69 165.1) (xy 193.04 165.1))
     (stroke (width 0) (type solid))
   )
@@
     )
   )
-  (symbol (lib_id "Jumper:Jumper_2_Open") (at 375.92 55.88 0) (unit 1)
+  (symbol (lib_id "Jumper:SolderJumper_2_Open") (at 375.92 55.88 0) (unit 1)
     (in_bom yes) (on_board yes) (dnp no) (fields_autoplaced)
     (property "Reference" "JP101" (at 375.92 49.53 0)
@@
       (effects (font (size 1.27 1.27)))
     )
-    (property "Footprint" "Connector_PinHeader_2.54mm:PinHeader_1x02_P2.54mm_Vertical" (at 375.92 55.88 0)
+    (property "Footprint" "Jumper:SolderJumper-2_P1.3mm_Open_RoundedPad1.0x1.5mm" (at 375.92 55.88 0)
       (effects (font (size 1.27 1.27)) hide)
     )
@@
     )
   )
-  (symbol (lib_id "Jumper:Jumper_2_Open") (at 196.85 165.1 0) (unit 1)
+  (symbol (lib_id "Jumper:SolderJumper_2_Open") (at 196.85 165.1 0) (unit 1)
     (in_bom yes) (on_board yes) (dnp no) (fields_autoplaced)
-    (property "Reference" "JP1" (at 196.85 158.75 0)
+    (property "Reference" "JP401" (at 196.85 158.75 0)
       (effects (font (size 1.27 1.27)))
     )
@@
       (effects (font (size 1.27 1.27)))
     )
-    (property "Footprint" "Connector_PinHeader_2.54mm:PinHeader_1x02_P2.54mm_Vertical" (at 196.85 165.1 0)
+    (property "Footprint" "Jumper:SolderJumper-2_P1.3mm_Open_RoundedPad1.0x1.5mm" (at 196.85 165.1 0)
       (effects (font (size 1.27 1.27)) hide)
     )
@@
       (project "DashShield"
         (path "/e63e39d7-6ac0-4ffd-8aa3-1841a4541b55"
-          (reference "JP1") (unit 1)
+          (reference "JP401") (unit 1)
         )
       )
@@
     )
   )
-  (symbol (lib_id "Jumper:Jumper_2_Open") (at 374.65 74.93 0) (unit 1)
+  (symbol (lib_id "Jumper:SolderJumper_2_Open") (at 374.65 74.93 0) (unit 1)
     (in_bom yes) (on_board yes) (dnp no) (fields_autoplaced)
     (property "Reference" "JP102" (at 374.65 68.58 0)
@@
       (effects (font (size 1.27 1.27)))
     )
-    (property "Footprint" "Connector_PinHeader_2.54mm:PinHeader_1x02_P2.54mm_Vertical" (at 374.65 74.93 0)
+    (property "Footprint" "Jumper:SolderJumper-2_P1.3mm_Open_RoundedPad1.0x1.5mm" (at 374.65 74.93 0)
       (effects (font (size 1.27 1.27)) hide)
     )
@@
     )
   )
-  (symbol (lib_id "Jumper:Jumper_2_Open") (at 375.92 132.08 0) (unit 1)
+  (symbol (lib_id "Jumper:SolderJumper_2_Open") (at 375.92 132.08 0) (unit 1)
     (in_bom yes) (on_board yes) (dnp no) (fields_autoplaced)
     (property "Reference" "JP201" (at 375.92 125.73 0)
@@
       (effects (font (size 1.27 1.27)))
     )
-    (property "Footprint" "Connector_PinHeader_2.54mm:PinHeader_1x02_P2.54mm_Vertical" (at 375.92 132.08 0)
+    (property "Footprint" "Jumper:SolderJumper-2_P1.3mm_Open_RoundedPad1.0x1.5mm" (at 375.92 132.08 0)
       (effects (font (size 1.27 1.27)) hide)
     )
@@
     )
   )
-  (symbol (lib_id "Jumper:Jumper_2_Open") (at 374.65 151.13 0) (unit 1)
+  (symbol (lib_id "Jumper:SolderJumper_2_Open") (at 374.65 151.13 0) (unit 1)
     (in_bom yes) (on_board yes) (dnp no) (fields_autoplaced)
     (property "Reference" "JP202" (at 374.65 144.78 0)
@@
       (effects (font (size 1.27 1.27)))
     )
-    (property "Footprint" "Connector_PinHeader_2.54mm:PinHeader_1x02_P2.54mm_Vertical" (at 374.65 151.13 0)
+    (property "Footprint" "Jumper:SolderJumper-2_P1.3mm_Open_RoundedPad1.0x1.5mm" (at 374.65 151.13 0)
       (effects (font (size 1.27 1.27)) hide)
     )

Commit message: feat: add ADC and data logger connector
Parts:
- removed D001, D005, D006: PMEG3050, Diode_SMD:D_SOD-128, symbol Device:D
- added C301, C302, C602: 10nF, Capacitor_SMD:C_0603_1608Metric, symbol Device:C
- added C601: 100nF, Capacitor_SMD:C_0603_1608Metric, symbol Device:C
- added D001, D005: PMEG100V080ELPD, Package_TO_SOT_SMD:Nexperia_CFP15_SOT-1289, symbol Diode:PMEG100V080ELPD
- added J002: Data Logger, Connector_Molex:Molex_Micro-Fit_3.0_43650-0315_1x03_P3.00mm_Vertical, symbol Connector_Generic:Conn_01x03
- added U601: ADS1015IDGS, Package_SO:TSSOP-10_3x3mm_P0.5mm, symbol Analog_ADC:ADS1015IDGS
- renumbered D007 to D006
Connections:
- net +3.3V: now also C601.1, C602.1, U601.8 (VDD)
- net +5V: now also J002.1 (Pin_1)
- net +BATT: now also D005.1 (A), D005.2 (A)
- net GND: now also C301.2, C302.2, C601.2, C602.2, J002.3 (Pin_3), U601.1 (ADDR), U601.3 (GND)
- net GPIO18/PCM.CLK: no longer R312.1
- net GPIO23: no longer R315.1
- net GPIO2/SDA1: now also U601.9 (SDA); no longer C004.1, R007.1, R008.2
- net GPIO3/SCL1: now also U601.10 (SCL); no longer C003.1, R005.1, R006.2
- net VS: now also D001.3 (K), D005.3 (K)
- net at J001.1 (Pin_1): now also D001.1 (A), D001.2 (A)
- new net TC Power Adjust: C302.1, R315.1, U601.6 (AIN2)
- new net VBATT Sense: C004.1, R007.1, R008.2, U601.4 (AIN0)
- new net VIN Sense: C003.1, J002.2 (Pin_2), R005.1, R006.2, U601.5 (AIN1)
- new net Wheel Slip Adjust: C301.1, R312.1, U601.7 (AIN3)
- no-connect marks 19 -> 22
Other:
- note added: "ADC"
- note added: "Data Logger Connection"
- note added: "Designed by Dallas Hart"
- moved on the sheet: C001, C002, C005, C006, C007, C401, D002, D003, D004, D006, J001, JP401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

Commit message: rev2
Connections:
- net FAST LED 0: now also J3.8 (Pin_8); no longer J3.6 (Pin_6)
- net FAST LED 1: now also J3.4 (Pin_4); no longer J3.7 (Pin_7)
- net FAST LED 2: now also J3.3 (Pin_3); no longer J3.8 (Pin_8)
- net SLOW LED 0: now also J3.6 (Pin_6); no longer J3.2 (Pin_2)
- net SLOW LED 1: now also J3.2 (Pin_2); no longer J3.3 (Pin_3)
- net SLOW LED 2: now also J3.7 (Pin_7); no longer J3.4 (Pin_4)
Changed lines of the file:
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@@
     (effects (font (size 1.27 1.27)) (justify right bottom))
   )
+  (label "SLOW LED 0" (at 184.15 29.21 180) (fields_autoplaced)
+    (effects (font (size 1.27 1.27)) (justify right bottom))
+  )
   (label "GPIO13{slash}PWM1" (at 31.75 69.85 0) (fields_autoplaced)
     (effects (font (size 1.27 1.27)) (justify left bottom))
@@
     (effects (font (size 1.27 1.27)) (justify right bottom))
   )
-  (label "SLOW LED 2" (at 148.59 34.29 0) (fields_autoplaced)
-    (effects (font (size 1.27 1.27)) (justify left bottom))
+  (label "SLOW LED 2" (at 184.15 31.75 180) (fields_autoplaced)
+    (effects (font (size 1.27 1.27)) (justify right bottom))
   )
   (label "FAST 1" (at 20.32 67.31 0) (fields_autoplaced)
@@
     (effects (font (size 1.27 1.27)) (justify right bottom))
   )
-  (label "FAST LED 1" (at 184.15 31.75 180) (fields_autoplaced)
-    (effects (font (size 1.27 1.27)) (justify right bottom))
-  )
   (label "TC LED 2" (at 285.75 204.47 180) (fields_autoplaced)
     (effects (font (size 1.27 1.27)) (justify right bottom))
@@
     (effects (font (size 1.27 1.27)) (justify right bottom))
   )
+  (label "FAST LED 1" (at 148.59 34.29 0) (fields_autoplaced)
+    (effects (font (size 1.27 1.27)) (justify left bottom))
+  )
   (label "TC LED 4" (at 267.97 204.47 180) (fields_autoplaced)
     (effects (font (size 1.27 1.27)) (justify right bottom))
@@
     (effects (font (size 1.27 1.27)) (justify left bottom))
   )
-  (label "TC LED 5" (at 262.89 190.5 0) (fields_autoplaced)
+  (label "FAST LED 2" (at 148.59 31.75 0) (fields_autoplaced)
     (effects (font (size 1.27 1.27)) (justify left bottom))
   )
-  (label "SLOW LED 1" (at 148.59 31.75 0) (fields_autoplaced)
+  (label "TC LED 5" (at 262.89 190.5 0) (fields_autoplaced)
     (effects (font (size 1.27 1.27)) (justify left bottom))
   )
+  (label "FAST LED 0" (at 184.15 34.29 180) (fields_autoplaced)
+    (effects (font (size 1.27 1.27)) (justify right bottom))
+  )
   (label "TC 1" (at 248.92 217.17 0) (fields_autoplaced)
     (effects (font (size 1.27 1.27)) (justify left bottom))
@@
     (effects (font (size 1.27 1.27)) (justify left bottom))
   )
-  (label "FAST LED 0" (at 184.15 29.21 180) (fields_autoplaced)
-    (effects (font (size 1.27 1.27)) (justify right bottom))
-  )
   (label "CAN1 High" (at 363.22 137.16 0) (fields_autoplaced)
     (effects (font (size 1.27 1.27)) (justify left bottom))
@@
     (effects (font (size 1.27 1.27)) (justify left bottom))
   )
-  (label "FAST LED 2" (at 184.15 34.29 180) (fields_autoplaced)
-    (effects (font (size 1.27 1.27)) (justify right bottom))
-  )
-  (label "SLOW LED 0" (at 148.59 29.21 0) (fields_autoplaced)
+  (label "SLOW LED 1" (at 148.59 29.21 0) (fields_autoplaced)
     (effects (font (size 1.27 1.27)) (justify left bottom))
   )
@@
       (effects (font (size 1.27 1.27) italic) hide)
     )
-    (property "Datasheet" "http://ww1.microchip.com/downloads/en/DeviceDoc/21801e.pdf" (at 273.05 148.59 0)
+    (property "Datasheet" "https://www.microchip.com/en-us/product/MCP2518FD#document-table" (at 273.05 148.59 0)
       (effects (font (size 1.27 1.27)) hide)
     )
@@
       (effects (font (size 1.27 1.27) italic) hide)
     )
-    (property "Datasheet" "http://ww1.microchip.com/downloads/en/DeviceDoc/21801e.pdf" (at 273.05 72.39 0)
+    (property "Datasheet" "https://www.microchip.com/en-us/product/MCP2518FD#document-table" (at 273.05 72.39 0)
       (effects (font (size 1.27 1.27)) hide)
     )
